File: phton_neopixel.brd (EAGLE design)
At the start: 39 x 59.7 mm, 13 parts, among them J1 Neopixel, J2 POWER_JACK, U2 PHOTON_WITH_HEADERS

Commit message: Changed pull-down resistor to 100k
Parts:
- R2: value 50k -> 100k
Changed lines of the file:
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@@
 </element>
 <element name="R1" library="resistor" package="0207/7" value="470" x="8.255" y="48.5775" rot="R90"/>
-<element name="R2" library="resistor" package="0207/7" value="50k" x="26.67" y="54.61"/>
+<element name="R2" library="resistor" package="0207/7" value="100k" x="26.67" y="54.61"/>
 <element name="U1" library="adafruit" package="TSSOP20" value="" x="6.35" y="38.1"/>
 <element name="U2" library="Spark" package="PHOTON" value="PHOTON_WITH_HEADERS" x="15.875" y="13.97" smashed="yes">
